File: KiCad/C64-PSU-PCB-replacement-for-902503-06.kicad_pcb (KiCad board)
At the start: 2 copper layers, 70.5 x 53.3 mm, 25 parts, among them J1 7V AC, J2 5,1V DC, J3 F-Mount, J4 F-Mount, U0 TO220_for_install

Commit message: Update C64-PSU-PCB-replacement-for-902503-06.kicad_pcb
Parts:
- C1: value 4700µF/16V -> 4700µF/25V
- J1: value 7V AC -> 7V-12V AC
- PS1: footprint SamacSys_Parts:OKRT15W12C -> C64-PSU-PCB-replacement-for-902503-06:OKRT15W12C
- renumbered REF** to +5.1V, REF** to GND
Connections:
- D1 pad 2: Net-(D1-Pad2) -> Net-(D1-A)
- D3 pad 1: Net-(D1-Pad2) -> Net-(D1-A)
- F2 pad 2: Net-(D1-Pad2) -> Net-(D1-A)
- J4 pad 2: Net-(D1-Pad2) -> (no net)
- PS1 pad 1: Net-(PS1-Pad1) -> unconnected-(PS1-REMOTE_ON/OFF_CONTROL-Pad1)
- U0 pad 1: Net-(U0-Pad1) -> unconnected-(U0-VI-Pad1)
- U0 pad 2: Net-(U0-Pad2) -> unconnected-(U0-GND-Pad2)
- U0 pad 3: Net-(U0-Pad3) -> unconnected-(U0-VO-Pad3)
Routing:
- net /+5,1V: track 179.9 -> 58.6 mm
- net Net-(D1-Pad2): track 51.3 -> 0.00 mm
- net Net-(D1-A): track 0.00 -> 51.3 mm
- net GND: track 183.6 -> 141.8 mm
- net Net-(D2-A): track 53.0 -> 31.8 mm
- net Net-(J1-Pin_2): track 56.3 -> 58.4 mm
Other:
- net class Default removed
